Commit message: added aruco node, and manipulation actions for testing box fit

File: sdl_packages/franka/multipanda_ros2/franka_description/robots/common/hand.xacro (robot description, xacro)
@@ -91,5 +91,5 @@
         <origin xyz="0 7.58e-3 45.25e-3" rpy="0 0 0" />
         <geometry>
-          <box size="17.5e-3 15.2e-3 18.5e-3" />
+          <box size="17.5e-3 15.2e-3 40.5e-3" />
         </geometry>
       </collision>
@@ -127,5 +127,5 @@
         <origin xyz="0 -7.58e-3 45.25e-3" rpy="0 0 0" />
         <geometry>
-          <box size="17.5e-3 15.2e-3 18.5e-3" />
+          <box size="17.5e-3 15.2e-3 40.5e-3" />
         </geometry>
       </collision>
